File: pcb/ym2610-pcb.kicad_pcb (KiCad board)
At the start: 4 copper layers, 100.9 x 77.5 mm, 132 parts, among them J1 MIDI_IN, J2 LINE_OUT, J3 HEADPHONES, J4 SPDIF_COAX, J5 UART, SW1 BTN_A, SW2 BTN_B, SW3 CRESET, U1 YM2610, U10 TSV914IPT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

Commit message: 1.0.0 of PCB as pictured in repo
Routing:
- removed copper zone on F.Cu, net GND
